Commit message: rotate axis 4 about 180 degree

File: kuka_kr210_support/urdf/kr210r2700extra_macro.xacro (robot description, xacro)
@@ -62,5 +62,5 @@
     <link name="${prefix}link_4">
       <visual>
-        <origin xyz="0 0 0" rpy="0 0 0"/>
+        <origin xyz="0 0 0" rpy="${180 * DEG2RAD} 0 0"/>
         <geometry>
           <mesh filename="package://kuka_kr210_support/meshes/kr210r2700extra/visual/link_4.dae" />
@@ -68,5 +68,5 @@
       </visual>
       <collision>
-        <origin xyz="0 0 0" rpy="0 0 0"/>
+        <origin xyz="0 0 0" rpy="${180 * DEG2RAD} 0 0"/>
         <geometry>
           <mesh filename="package://kuka_kr210_support/meshes/kr210r2700extra/collision/link_4.stl" />
